File: S3G4_LAB_rev2.1/04_esquematicos/kicad/ch3.kicad_sch (KiCad schematic)
At the start: 0 parts

Commit message: S10: CH2 y CH3 dibujados en sus hojas (filtro 1 MHz, textos reposicionados)
Co-Authored-By: Claude Sonnet 5.5 <noreply@anthropic.com>
Parts:
- added C301: 20pF 2% C0G 250V, Capacitor_SMD:C_0603_1608Metric, symbol Device:C
- added C302: 15pF 2% C0G 250V, Capacitor_SMD:C_0805_2012Metric, symbol Device:C
- added C303: DNP, Capacitor_SMD:C_0603_1608Metric, symbol Device:C
- added C304: 1nF 1% C0G, Capacitor_SMD:C_0603_1608Metric, symbol Device:C
- added C305: 68pF 5% C0G, Capacitor_SMD:C_0603_1608Metric, symbol Device:C
- added C306: 1.2nF C0G 200V, Capacitor_SMD:C_1206_3216Metric, symbol Device:C
- added C307: ~8.7pF C0G 200V, Capacitor_SMD:C_1206_3216Metric, symbol Device:C
- added C308: 1.8nF C0G 50V, Capacitor_SMD:C_0603_1608Metric, symbol Device:C
- added C309, C312: 56pF C0G, Capacitor_SMD:C_0603_1608Metric, symbol Device:C
- added C310: 47pF C0G, Capacitor_SMD:C_0603_1608Metric, symbol Device:C
- added C311: 220pF C0G, Capacitor_SMD:C_0603_1608Metric, symbol Device:C
- added C313: 1pF C0G, Capacitor_SMD:C_0603_1608Metric, symbol Device:C
- added C314: 1uF, Capacitor_SMD:C_0603_1608Metric, symbol Device:C
- added C315: 470pF C0G, Capacitor_SMD:C_0603_1608Metric, symbol Device:C
- added C316, C317, C318, C319, C320, C321, C322, C323, C324: 100nF X7R 16V, Capacitor_SMD:C_0402_1005Metric, symbol Device:C
- added C325, C326: 10uF X5R 25V, Capacitor_SMD:C_0805_2012Metric, symbol Device:C
- added D301: BAV199, Package_TO_SOT_SMD:SOT-23, symbol Diode:BAV99
- added D302, D303: BAV99, Package_TO_SOT_SMD:SOT-23, symbol Diode:BAV99
- added D304: 1N4148W, Diode_SMD:D_SOD-123, symbol Diode:1N4148W
- added J301: BNC, s3g4:BNC_Kinghelm_KH-BNC50-3511_Horizontal, symbol Connector:Conn_Coaxial
- added K301: TQ2SA-5V-Z, s3g4:Relay_Panasonic_TQ2SA_SMD, symbol s3g4:TQ2SA-5V-Z
- added Q301: 2N7002, Package_TO_SOT_SMD:SOT-23, symbol Transistor_FET:2N7002
- added R301, R302: 549k 0.1%, Resistor_SMD:R_1206_3216Metric, symbol Device:R
- added R303: 11.0k 0.1%, Resistor_SMD:R_0805_2012Metric, symbol Device:R
- added R304, R305: 49.9k, Resistor_SMD:R_1206_3216Metric, symbol Device:R
- added R306: 10M, Resistor_SMD:R_1206_3216Metric, symbol Device:R
- added R307: 10M 1%, Resistor_SMD:R_0603_1608Metric, symbol Device:R
- added R308, R309, R337: 1k, Resistor_SMD:R_0603_1608Metric, symbol Device:R
- added R310, R319, R322: 270, Resistor_SMD:R_0603_1608Metric, symbol Device:R
- added R311: 150 1%, Resistor_SMD:R_0603_1608Metric, symbol Device:R
- added R312: 49.9 1%, Resistor_SMD:R_0603_1608Metric, symbol Device:R
- added R313, R314, R343, R344: 49.9, Resistor_SMD:R_0603_1608Metric, symbol Device:R
- added R315: 12.4k 0.1%, Resistor_SMD:R_0402_1005Metric, symbol Device:R
- added R316: 100 0.1%, Resistor_SMD:R_0402_1005Metric, symbol Device:R
- added R317, R320: 470, Resistor_SMD:R_0603_1608Metric, symbol Device:R
- added R318: 1.00k 1%, Resistor_SMD:R_0603_1608Metric, symbol Device:R
- added R321, R323, R324: 2.2k, Resistor_SMD:R_0603_1608Metric, symbol Device:R
- added R325, R326: 1.1k, Resistor_SMD:R_0603_1608Metric, symbol Device:R
- added R327, R329, R330: 10.0k 1%, Resistor_SMD:R_0603_1608Metric, symbol Device:R
- added R328: 7.5k, Resistor_SMD:R_0603_1608Metric, symbol Device:R
- added R331: 5.1k, Resistor_SMD:R_0603_1608Metric, symbol Device:R
- added R332, R345: 68, Resistor_SMD:R_0603_1608Metric, symbol Device:R
- added R333, R334: 10k 1%, Resistor_SMD:R_0603_1608Metric, symbol Device:R
- added R335: 100, Resistor_SMD:R_0603_1608Metric, symbol Device:R
- added R336: 100k, Resistor_SMD:R_0603_1608Metric, symbol Device:R
- added R340, R341, R342: 3.3k, Resistor_SMD:R_0603_1608Metric, symbol Device:R
- added R346: 560, Resistor_SMD:R_0603_1608Metric, symbol Device:R
- added R347: 120, Resistor_SMD:R_0603_1608Metric, symbol Device:R
- added R348, R349: 150, Resistor_SMD:R_0603_1608Metric, symbol Device:R
- added SW301: SS23H37L6, s3g4:SW_Slide_DP3T_XKB_SS23H37, symbol s3g4:SS23H37L6
- added U301: OPA810IDBVR, Package_TO_SOT_SMD:SOT-23-5, symbol Amplifier_Operational:OPA810xDBV
- added U302: 74HC4051D, Package_SO:SOIC-16_3.9x9.9mm_P1.27mm, symbol 74xx:74HC4051
- added U303, U305: AD8039ARZ-REEL7, Package_SO:SOIC-8_3.9x4.9mm_P1.27mm, symbol Amplifier_Operational:LM6172
- added U306: OPA836IDBVR, Package_TO_SOT_SMD:SOT-23-6, symbol Amplifier_Operational:ADA4807-1
- added VC301: 2-6pF, s3g4:C_Trimmer_SEHWA_STC3MA06_3.2x4.5mm, symbol Device:C_Trim
Connections:
- new net +3V3: R333.1, R334.1
- new net +AFE_4V9: C316.1, C318.1, C320.1, C322.1, C325.1, D301.2 (A), U301.5 (V+), U302.16 (VCC), U303.8 (V+), U305.8 (V+)
- new net -AFE_4V9: C317.1, C319.1, C321.1, C323.1, C326.2, D301.1 (K), U301.2 (V-), U302.7 (VEE), U303.4 (V-), U305.4 (V-)
- new net AGND: C304.2, C305.2, C307.2, C310.2, C312.2, C314.1, C315.2, C316.2, C317.2, C318.2, C319.2, C320.2, C321.2, C322.2, C323.2, C324.2, C325.2, C326.1, J301.2 (Ext), R303.2, R306.2, R307.2, R314.2, R316.2, R319.1, R322.1, R341.1, R342.1, R344.2, R347.2, SW301.3 (T2), U302.2 (A6), U302.6 (~{E}), U302.8 (GND), U306.2 (V-)
- new net CH3_AC: C308.2, SW301.1 (T1)
- new net CH3_ADC: C315.1, R332.2
- new net CH3_BNC: C301.1, C306.1, J301.1 (In), R301.1, R304.1
- new net CH3_BUF_INP: R308.2, U301.3 (+)
- new net CH3_BUF_OUT: R309.1, R337.1, U301.1, U301.4 (-), U302.13 (A0)
- new net CH3_CPL_A: R333.2, SW301.5 (T1)
- new net CH3_CPL_B: R334.2, SW301.8 (T3)
- new net CH3_CPL_COM: R307.1, R308.1, SW301.2 (COM)
- new net CH3_DIV_MID: C301.2, C302.1, C303.1, R301.2, R302.1, VC301.1
- new net CH3_DRV_OUT: C313.2, R329.2, R332.1, U306.1
- new net CH3_EQ: C307.1, K301.9 (NC), R306.1
- new net CH3_F1_A: R323.2, R348.1
- new net CH3_F1_B: R324.2, R349.1
- new net CH3_F1_INP: C310.1, R349.2, U305.3 (+)
- new net CH3_F1_MID: C309.1, R324.1, R348.2
- new net CH3_F1_OUT: C309.2, R325.1, U305.1, U305.2 (-)
- new net CH3_F2_INP: C312.1, R326.2, U305.5 (+)
- new net CH3_F2_MID: C311.1, R325.2, R326.1
- new net CH3_FILT_OUT: C311.2, R327.1, U305.6 (-), U305.7
- new net CH3_G1_INN: D302.3 (K), R318.1, R319.2, R341.2, U303.2 (-)
- new net CH3_G1_INP: D302.1 (K), D302.2 (A), R317.2, U303.3 (+)
- new net CH3_G1_OUT: R318.2, R320.1, U303.1
- new net CH3_G2_INN: D303.3 (K), R322.2, R342.2, R345.1, U303.6 (-)
- new net CH3_G2_INP: D303.1 (K), D303.2 (A), R320.2, U303.5 (+)
- new net CH3_G2_OUT: R321.2, R323.1, U303.7
- new net CH3_K_COIL_N: D304.2 (A), K301.10 (-), Q301.3 (D)
- new net CH3_K_CTRL: R335.1
- new net CH3_K_GATE: Q301.1 (G), R335.2, R336.2
- new net CH3_LAD1: R309.2, R310.1, R337.2, R340.1, U302.14 (A1)
- new net CH3_LAD2: R310.2, R311.1, R340.2, U302.15 (A2)
- new net CH3_LAD3: R311.2, R312.1, U302.12 (A3)
- new net CH3_LAD4: R312.2, R313.1, R343.1, U302.1 (A4)
- new net CH3_LAD5: R313.2, R314.1, R343.2, R344.1, U302.5 (A5)
- new net CH3_MUX_OUT: R317.1, U302.3 (A)
- new net CH3_OFFSET_DAC: R328.1
- new net CH3_RF2_MID: R321.1, R345.2
- new net CH3_ROFF_MID: R328.2, R346.1
- new net CH3_RS_MID: R304.2, R305.1
- new net CH3_SEL: C308.1, D301.3 (K), K301.3 (COM), SW301.4 (T3)
- new net CH3_SENSEL_A: U302.11 (S0)
- new net CH3_SENSEL_B: U302.10 (S1)
- new net CH3_SENSEL_C: U302.9 (S2)
- new net CH3_SUM: C313.1, R327.2, R329.1, R346.2, U306.4 (-)
- new net CH3_TAP: C302.2, C303.2, C304.1, C305.1, K301.2 (NC), R302.2, R303.1, VC301.2
- new net CH3_VCHECK: R315.2, R316.1, U302.4 (A7)
- new net CH3_VMID: C314.2, R330.2, R331.1, U306.3 (+)
- new net CH3_VMID_LO: R331.2, R347.1
- new net CH3_X1: C306.2, K301.4 (NO), K301.8 (COM), R305.2
- new net GND: Q301.2 (S), R336.1, SW301.6 (COM)
- new net RELAY_COM: D304.1 (K), K301.1 (+)
- new net VDDA: C324.1, U306.5 (~{DISABLE}), U306.6 (V+)
- new net VREF_2V5: R315.1, R330.1
- no-connect marks 0 -> 2
Other:
- note added: "1 · Entrada: J301, divisor ÷100, rama ×1 y réplica"
- note added: "2 · Relé K301 TQ2SA-5V-Z, reposo = ÷100"
- note added: "3 · Sujeción D301, acoplo SW301, C_AC, R_BIAS y R_PROT"
- note added: "4 · Buffer U301"
- note added: "5 · Escalera, VCHECK y U302"
- note added: "6 · Ganancia ×50 U303A ×5.016, U303B ×10.08, R_SER y BAV99"
- note added: "7 · Filtro anti-alias U305 a 1 MHz (dos Sallen-Key)"
- note added: "8 · Etapa final U306, VMID y red del pin (CH3_ADC → ADC4, pin por fijar)"
- note added: "9 · Driver del relé (Q301, D304, R335, R336) La corriente de la bobina vuelve por GND, no por AGND."
- note added: "ABIERTO (§5 de CH1_PIEZAS_Y_REDES.md y §4 de CH23_PIEZAS_Y_REDES.md), no dibujado: - Circuito común del economizador (P-MOSFET de arranque, Schottky desde 3.3 V, línea RELAY_KICK): va en la hoja de control/alimentación, no en la de CH3. - TVS de riel: es de la hoja de alimentación, no de CH3. - El 74HC165 que lee CH3_CPL_A/B cuelga del STM32, en el bus de los 74HCT595. - Partición AGND/GND: la de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"
