File: S3G4_LAB_rev2.1/04_esquematicos/kicad/s3g4.kicad_sch (KiCad schematic)
At the start: 89 parts, among them J101 BNC, K101 TQ2SA-5V-Z, Q101 2N7002, SW101 SS23H37L6, U101 OPA810IDBVR, U102 74HC4051D, U103 AD8039ARZ-REEL7, U105 AD8039ARZ-REEL7, U106 OPA836IDBVR

Commit message: S10: hojas CH2 y CH3 en la raíz y CH2 dibujado (copia de CH1 con filtro a 1 MHz)
Co-Authored-By: Claude Sonnet 5.5 <noreply@anthropic.com>
Other:
- added sheet CH2 (ch2.kicad_sch)
- added sheet CH3 (ch3.kicad_sch)
Changed lines of the file:
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@@
 		)
 	)
+	(sheet
+    (at 500 50)
+    (size 40 25)
+    (exclude_from_sim no)
+    (in_bom yes)
+    (on_board yes)
+    (dnp no)
+    (fields_autoplaced yes)
+    (stroke (width 0.1524) (type solid))
+    (fill (color 0 0 0 0.0))
+    (property "Sheetname" "CH2"
+      (at 500 49.365 0)
+      (show_name no)
+      (do_not_autoplace no)
+      (effects (font (size 1.27 1.27)) (justify left bottom))
+    )
+    (property "Sheetfile" "ch2.kicad_sch"
+      (at 500 75.635 0)
+      (show_name no)
+      (do_not_autoplace no)
+      (effects (font (size 1.27 1.27)) (justify left top))
+    )
+    (instances
+      (project "s3g4"
+        (path "/de82ce61-fda9-4439-b3fa-fd2016785b6d" (page "2"))
+      )
+    )
+  )
+	(sheet
+    (at 500 90)
+    (size 40 25)
+    (exclude_from_sim no)
+    (in_bom yes)
+    (on_board yes)
+    (dnp no)
+    (fields_autoplaced yes)
+    (stroke (width 0.1524) (type solid))
+    (fill (color 0 0 0 0.0))
+    (property "Sheetname" "CH3"
+      (at 500 89.365 0)
+      (show_name no)
+      (do_not_autoplace no)
+      (effects (font (size 1.27 1.27)) (justify left bottom))
+    )
+    (property "Sheetfile" "ch3.kicad_sch"
+      (at 500 115.635 0)
+      (show_name no)
+      (do_not_autoplace no)
+      (effects (font (size 1.27 1.27)) (justify left top))
+    )
+    (instances
+      (project "s3g4"
+        (path "/de82ce61-fda9-4439-b3fa-fd2016785b6d" (page "3"))
+      )
+    )
+  )
 	(sheet_instances
 		(path "/"
